Commit message: updated colors of lwa4p

File: schunk_description/urdf/lwa4d/lwa4d.urdf.xacro (robot description, xacro)
@@ -156,5 +156,5 @@
       <parent link="${name}_4_link"/>
       <child link="${name}_5_link"/>
-      <axis xyz="0 0 1"/>
+      <axis xyz="0 0 -1"/>
       <limit effort="20.7" velocity="0.43633" lower="${-M_PI + safety_offset}" upper="${M_PI - safety_offset}"/>
     </joint>

File: schunk_description/urdf/lwa4p/lwa4p.gazebo.xacro (robot description, xacro)
@@ -2,33 +2,28 @@
 <robot xmlns:xacro="http://www.ros.org/wiki/xacro">
   <xacro:macro name="schunk_lwa4p_gazebo" params="name">
-    <gazebo reference="${name}_0_link">
+    <gazebo reference="${name}_1_link">
       <gravity>true</gravity>
       <self_collide>false</self_collide>
       <material value="Schunk/LightGrey" />
     </gazebo>
-    <gazebo reference="${name}_1_link">
+    <gazebo reference="${name}_2_link">
       <gravity>true</gravity>
       <self_collide>false</self_collide>
       <material value="Schunk/Blue" />
     </gazebo>
-    <gazebo reference="${name}_2_link">
+    <gazebo reference="${name}_3_link">
       <gravity>true</gravity>
       <self_collide>false</self_collide>
       <material value="Schunk/LightGrey" />
     </gazebo>
-    <gazebo reference="${name}_3_link">
+    <gazebo reference="${name}_4_link">
       <gravity>true</gravity>
       <self_collide>false</self_collide>
       <material value="Schunk/Blue" />
     </gazebo>
-    <gazebo reference="${name}_4_link">
+    <gazebo reference="${name}_5_link">
       <gravity>true</gravity>
       <self_collide>false</self_collide>
       <material value="Schunk/LightGrey" />
-    </gazebo>
-    <gazebo reference="${name}_5_link">
-      <gravity>true</gravity>
-      <self_collide>false</self_collide>
-      <material value="Schunk/Blue" />
     </gazebo>
     <gazebo reference="${name}_6_link">

File: schunk_description/urdf/lwa4p/lwa4p.urdf.xacro (robot description, xacro)
@@ -67,5 +67,5 @@
           <mesh filename="package://schunk_description/meshes/lwa4p/arm_1_link.stl" />
         </geometry>
-        <material name="Schunk/Blue" />
+        <material name="Schunk/LightGrey" />
       </visual>
       <collision>
@@ -99,5 +99,5 @@
           <mesh filename="package://schunk_description/meshes/lwa4p/arm_2_link.stl" />
         </geometry>
-        <material name="Schunk/LightGrey" />
+        <material name="Schunk/Blue" />
       </visual>
       <collision>
@@ -131,5 +131,5 @@
           <mesh filename="package://schunk_description/meshes/lwa4p/arm_3_link.stl" />
         </geometry>
-        <material name="Schunk/Blue" />
+        <material name="Schunk/LightGrey" />
       </visual>
       <collision>
@@ -163,5 +163,5 @@
           <mesh filename="package://schunk_description/meshes/lwa4p/arm_4_link.stl" />
         </geometry>
-        <material name="Schunk/LightGrey" />
+        <material name="Schunk/Blue" />
       </visual>
       <collision>
@@ -195,5 +195,5 @@
           <mesh filename="package://schunk_description/meshes/lwa4p/arm_5_link.stl" />
         </geometry>
-        <material name="Schunk/Blue" />
+        <material name="Schunk/LightGrey" />
       </visual>
       <collision>
